File: pcb/KiCad/Input_Output_Section.kicad_sch (KiCad schematic)
At the start: 68 parts, among them J10 Ref_In_2, J11 Ctrl_Out_1, J12 Ctrl_In_2, J13 PD_Mon_2, J14 Ctrl_Out_2, J15 Diff_Out_2, J17 Diff_Mon_1, J18 Diff_Mon_2, J3 PD_In_1, J5 Diff_Out_1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

Commit message: Fixed trailing whitespace in MFN
Parts:
- SW2: MFN Omron Electronics -> Omron Electronics
Changed lines of the file:
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@@
       (effects (font (size 1.27 1.27)) hide)
     )
-    (property "MFN" "Omron Electronics " (at 166.37 129.54 0)
+    (property "MFN" "Omron Electronics" (at 166.37 129.54 0)
       (effects (font (size 1.27 1.27)) hide)
     )
